File: PCB Design/Color sensor_LED Board.brd (EAGLE design)
At the start: 20 x 20 mm, 25 parts, among them U1 2DD2656-7

Commit message: corrected unconnected traces and IR LED problem
Parts:
- moved R13 14.9 mm to (-0.64, -7.62), flipped to the top, turned to 96.7 degrees
- moved LED10 13.6 mm to (-3.05, -6.60), turned to 146.2 degrees
- moved R1 3.22 mm to (3.30, -7.87), turned to 24.3 degrees
- moved R4 2.32 mm to (2.41, -5.84), turned to 23.8 degrees
Connections:
- net GND: now also LED10.C
- net N$15: no longer LED10.C
Routing:
- net VCC: track 53.0 -> 59.0 mm
- net GND: track 16.6 -> 20.7 mm, vias 0 -> 1
- net N$6: track 6.71 -> 3.60 mm
- net N$12: track 4.18 -> 1.90 mm
- net N$17: track 4.09 -> 1.98 mm, vias 1 -> 0
- net N$15: track 40.9 -> 38.9 mm
Other:
- board text added: "COLOR SENSOR LED MODULE"
